Commit message: adding servo motors to existing file

File: src/arm_teleop/urdf/simple_arm.urdf (robot description, URDF)
Before this commit: robot simple_arm, 4 links, 3 joints
Links:
- added link claw_servo; visual box size=0.06 0.04 0.03
- added link elbow_servo; visual cylinder length=0.05 radius=0.035
- added link shoulder_servo; visual cylinder length=0.05 radius=0.04
Joints:
- added joint base_to_shoulder_servo: type fixed, parent base_link, child shoulder_servo, origin xyz=0 0 0.05 rpy=0 0 0
- added joint forearm_to_claw_servo: type fixed, parent forearm, child claw_servo, origin xyz=0 0 0.125 rpy=0 0 0
- added joint upper_arm_to_elbow_servo: type fixed, parent upper_arm, child elbow_servo, origin xyz=0 0 0.15 rpy=0 0 0
- joint claw_joint: origin xyz=0 0 0.125 rpy=0 0 0 -> xyz=0 0 0.015 rpy=0 0 0; parent forearm -> claw_servo
- joint elbow_joint: origin xyz=0 0 0.15 rpy=0 0 0 -> xyz=0 0 0.025 rpy=0 0 0; parent upper_arm -> elbow_servo
- joint shoulder_joint: origin xyz=0 0 0.05 rpy=0 0 0 -> xyz=0 0 0.025 rpy=0 0 0; parent base_link -> shoulder_servo

Commit message: changing measurements

File: src/arm_teleop/urdf/simple_arm.urdf (robot description, URDF)
Before this commit: robot simple_arm, 7 links, 6 joints
Links:
- link base_link: geometry visual cylinder length=0.05 radius=0.08
- link forearm: geometry visual box size=0.045 0.045 0.22
- link shoulder_servo: geometry visual cylinder length=0.06 radius=0.04
- link upper_arm: geometry visual box size=0.05 0.05 0.25
Joints:
- joint claw_joint: limit lower=0.0 upper=0.1 effort=5 velocity=0.5 -> lower=0.0 upper=0.05 effort=5 velocity=0.5; origin xyz=0 0 0.015 rpy=0 0 0 -> xyz=0 0 0.02 rpy=0 0 0
- joint elbow_joint: limit lower=0.0 upper=2.62 effort=10 velocity=1.0 -> lower=0.0 upper=2.0 effort=10 velocity=1.0
- joint forearm_to_claw_servo: origin xyz=0 0 0.125 rpy=0 0 0 -> xyz=0 0 0.22 rpy=0 0 0
- joint shoulder_joint: limit lower=-3.14 upper=3.14 effort=10 velocity=1.0 -> lower=-1.57 upper=1.57 effort=10 velocity=1.0; origin xyz=0 0 0.025 rpy=0 0 0 -> xyz=0 0 0.03 rpy=0 0 0
- joint upper_arm_to_elbow_servo: origin xyz=0 0 0.15 rpy=0 0 0 -> xyz=0 0 0.25 rpy=0 0 0

Commit message: working arm with servo motor and elbow colored.

File: src/arm_teleop/urdf/simple_arm.urdf (robot description, URDF)
Before this commit: robot simple_arm, 7 links, 6 joints
Links:
- removed link claw
- removed link claw_servo
- removed link elbow_servo
- removed link forearm
- removed link shoulder_servo
- removed link upper_arm
- added link elbow_link; visual cylinder length=0.06 radius=0.03
- added link forearm_link; visual box size=0.04 0.04 0.25
- added link gripper_link; visual box size=0.06 0.04 0.04
- added link shoulder_link; visual cylinder length=0.08 radius=0.05
- added link upper_arm_link; visual box size=0.05 0.05 0.3
- link base_link: geometry visual cylinder length=0.05 radius=0.1
Joints:
- removed joint base_to_shoulder_servo
- removed joint claw_joint
- removed joint elbow_joint
- removed joint forearm_to_claw_servo
- removed joint shoulder_joint
- removed joint upper_arm_to_elbow_servo
- added joint base_to_shoulder: type fixed, parent base_link, child shoulder_link, origin xyz=0 0 0.05 rpy=0 0 0
- added joint elbow_to_forearm: type revolute, parent elbow_link, child forearm_link, origin xyz=0 0 0.06 rpy=0 0 0, axis 0 1 0, limit lower=-1.57 upper=1.57 effort=10 velocity=1
- added joint forearm_to_gripper: type fixed, parent forearm_link, child gripper_link, origin xyz=0 0 0.25 rpy=0 0 0
- added joint shoulder_to_upper_arm: type revolute, parent shoulder_link, child upper_arm_link, origin xyz=0 0 0.08 rpy=0 0 0, axis 0 1 0, limit lower=-1.57 upper=1.57 effort=10 velocity=1
- added joint upper_arm_to_elbow: type fixed, parent upper_arm_link, child elbow_link, origin xyz=0 0 0.3 rpy=0 0 0

Commit message: changing file so that arm opens directly.

File: src/arm_teleop/urdf/simple_arm.urdf (robot description, URDF)
Before this commit: robot colored_arm, 6 links, 5 joints
Links:
- removed link gripper_link
- added link claw_base_link; visual box size=0.05 0.05 0.02
- added link claw_left_link; visual box size=0.02 0.05 0.08
- added link claw_right_link; visual box size=0.02 0.05 0.08
- added link wrist_link; visual cylinder length=0.05 radius=0.025
Joints:
- removed joint forearm_to_gripper
- added joint claw_base_to_left: type revolute, parent claw_base_link, child claw_left_link, origin xyz=0.025 0 0.01 rpy=0 0 0, axis 0 1 0, limit lower=0 upper=0.6 effort=2 velocity=1
- added joint claw_base_to_right: type revolute, parent claw_base_link, child claw_right_link, origin xyz=-0.025 0 0.01 rpy=0 0 0, axis 0 1 0, limit lower=-0.6 upper=0 effort=2 velocity=1
- added joint forearm_to_wrist: type revolute, parent forearm_link, child wrist_link, origin xyz=0 0 0.25 rpy=0 0 0, axis 0 0 1, limit lower=-1.57 upper=1.57 effort=5 velocity=1
- added joint wrist_to_claw_base: type fixed, parent wrist_link, child claw_base_link, origin xyz=0 0 0.05 rpy=0 0 0
